Commit message: pybullet testing

File: descriptions/urdf/gx7.urdf (robot description, URDF)
Before this commit: robot GX7_250721, 9 links, 8 joints
Links:
- link Link7: mass 0 -> 0.01
Joints:
- joint base_joint: origin xyz=0 0 0 rpy=0 -1.5708 0 -> xyz=0 0 0 rpy=0 -1.5707963 0
- joint joint1: origin xyz=0.0695 0 0 rpy=1.5708 0 1.5708 -> xyz=0.0695 0 0 rpy=1.5707963 0 1.5707963
- joint joint2: limit lower=0 upper=3.1415 effort=5 velocity=3.2 -> lower=0 upper=3.141592615 effort=5 velocity=3.2; origin xyz=0 0.0235 0.05 rpy=1.5708 -1.5708 3.14 -> xyz=0 0.0235 0.05 rpy=1.5707963 -1.5707963 3.1415926
- joint joint3: origin xyz=0 -0.1105 -0.0235 rpy=1.5708 0 0 -> xyz=0 -0.1105 -0.0235 rpy=1.5707963 0 0
- joint joint4: limit lower=0 upper=3.1415 effort=5 velocity=3.2 -> lower=0 upper=3.141592615 effort=5 velocity=3.2; origin xyz=0.077 0.0235 0.21049 rpy=-1.5708 0 0 -> xyz=0.077 0.0235 0.21049 rpy=-1.5707963 0 0
- joint joint5: origin xyz=0 0.217 -0.0235 rpy=-1.5708 0 0 -> xyz=0 0.217 -0.0235 rpy=-1.5707963 0 0
- joint joint6: limit lower=-1.5708 upper=1.5708 effort=5 velocity=3.2 -> lower=-1.5707963 upper=1.5707963 effort=5 velocity=3.2; origin xyz=0 0.013 0.05 rpy=1.5708 0 0 -> xyz=0 0.013 0.05 rpy=1.5707963 0 0
- joint joint7: limit lower=-3.1415 upper=3.1415 effort=5 velocity=3.2 -> lower=-3.141592615 upper=3.141592615 effort=5 velocity=3.2; origin xyz=0 0.099 0.013 rpy=1.5708 0 -3.1416 -> xyz=0 0.099 0.013 rpy=1.5707963 0 -3.141592616

Commit message: not finishing

File: descriptions/urdf/gx7.urdf (robot description, URDF)
Before this commit: robot GX7_250721, 9 links, 8 joints
Joints:
- joint joint7: limit lower=-3.141592615 upper=3.141592615 effort=5 velocity=3.2 -> (none); type revolute -> fixed
